File: espixelstick/espixelstick.kicad_pcb (KiCad board)
At the start: 2 copper layers, 36.8 x 15.2 mm, 11 parts

Commit message: update to kicad7
Connections:
- esp1 pad 5: Net-(esp1-Pad5) -> unconnected-(esp1-RST-Pad5)
Other:
- net class Default removed

Commit message: add 7.0 files, fix missing symbols
Parts:
- capa2: value capa2 -> C_Polarized
- connector1: value connector1 -> Conn_01x04_Pin
Changed lines of the file:
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@@
     (descr "https://www.omron.com/ecb/products/pdf/en-b3f.pdf")
     (tags "tact sw push 6mm")
-    (property "Sheetfile" "C:/programming_land/kicad_projects/kp_espixelstick/espixelstick/espixelstick.sch")
+    (property "Sheetfile" "espixelstick.kicad_sch")
     (property "Sheetname" "")
     (property "ki_description" "Push button switch, generic, two pins")
@@
     (descr "C, Disc series, Radial, pin pitch=2.50mm, , diameter*width=3.0*1.6mm^2, Capacitor, http://www.vishay.com/docs/45233/krseries.pdf")
     (tags "C Disc series Radial pin pitch 2.50mm  diameter 3.0mm width 1.6mm Capacitor")
-    (property "Sheetfile" "C:/programming_land/kicad_projects/kp_espixelstick/espixelstick/espixelstick.sch")
+    (property "Sheetfile" "espixelstick.kicad_sch")
     (property "Sheetname" "")
     (property "ki_description" "Unpolarized capacitor, small symbol")
@@
     (descr "CP, Radial series, Radial, pin pitch=2.00mm, , diameter=5mm, Electrolytic Capacitor")
     (tags "CP Radial series Radial pin pitch 2.00mm  diameter 5mm Electrolytic Capacitor")
-    (property "Sheetfile" "C:/programming_land/kicad_projects/kp_espixelstick/espixelstick/espixelstick.sch")
-    (property "Sheetname" "")
+    (property "Sheetfile" "espixelstick.kicad_sch")
+    (property "Sheetname" "")
+    (property "ki_description" "Polarized capacitor")
+    (property "ki_keywords" "cap capacitor")
     (attr through_hole)
     (fp_text reference "capa2" (at 1 -3.81 90) (layer "F.SilkS")
         (effects (font (size 1 1) (thickness 0.15)))
     )
-    (fp_text value "capa2" (at 1 3.81 90) (layer "F.Fab")
+    (fp_text value "C_Polarized" (at 1 3.81 90) (layer "F.Fab")
         (effects (font (size 1 1) (thickness 0.15)))
     )
@@
     (descr "Through hole straight pin header, 1x04, 2.54mm pitch, single row")
     (tags "Through hole pin header THT 1x04 2.54mm single row")
-    (property "Sheetfile" "C:/programming_land/kicad_projects/kp_espixelstick/espixelstick/espixelstick.sch")
-    (property "Sheetname" "")
+    (property "Sheetfile" "espixelstick.kicad_sch")
+    (property "Sheetname" "")
+    (property "ki_description" "Generic connector, single row, 01x04, script generated")
+    (property "ki_keywords" "connector")
     (attr through_hole)
     (fp_text reference "connector1" (at 0 -2.33 90) (layer "F.SilkS")
         (effects (font (size 1 1) (thickness 0.15)))
     )
-    (fp_text value "connector1" (at 0 9.95 90) (layer "F.Fab")
+    (fp_text value "Conn_01x04_Pin" (at 0 9.95 90) (layer "F.Fab")
         (effects (font (size 1 1) (thickness 0.15)))
     )
@@
     (descr "D, DO-35_SOD27 series, Axial, Horizontal, pin pitch=7.62mm, , length*diameter=4*2mm^2, , http://www.diodes.com/_files/packages/DO-35.pdf")
     (tags "D DO-35_SOD27 series Axial Horizontal pin pitch 7.62mm  length 4mm diameter 2mm")
-    (property "Sheetfile" "C:/programming_land/kicad_projects/kp_espixelstick/espixelstick/espixelstick.sch")
+    (property "Sheetfile" "espixelstick.kicad_sch")
     (property "Sheetname" "")
     (property "ki_description" "Diode")
@@
     (descr "Module, ESP-8266, ESP-01, 8 pin")
     (tags "Module ESP-8266 ESP8266")
-    (property "Sheetfile" "C:/programming_land/kicad_projects/kp_espixelstick/espixelstick/espixelstick.sch")
+    (property "Sheetfile" "espixelstick.kicad_sch")
     (property "Sheetname" "")
     (property "ki_description" "ESP8266 ESP-01 module, v090")
@@
     (descr "TO-92 leads in-line, wide, drill 0.8mm (see NXP sot054_po.pdf)")
     (tags "to-92 sc-43 sc-43a sot54 PA33 transistor")
-    (property "Sheetfile" "C:/programming_land/kicad_projects/kp_espixelstick/espixelstick/espixelstick.sch")
+    (property "Sheetfile" "espixelstick.kicad_sch")
     (property "Sheetname" "")
     (property "ki_description" "0.2A Id, 200V Vds, N-Channel MOSFET, 2.6V Logic Level, TO-92")
@@
     (descr "Through hole straight pin header, 1x02, 2.54mm pitch, single row")
     (tags "Through hole pin header THT 1x02 2.54mm single row")
-    (property "Sheetfile" "C:/programming_land/kicad_projects/kp_espixelstick/espixelstick/espixelstick.sch")
+    (property "Sheetfile" "espixelstick.kicad_sch")
     (property "Sheetname" "")
     (property "ki_description" "Generic connector, single row, 01x02, script generated (kicad-library-utils/schlib/autogen/connector/)")
@@
     (descr "Resistor, Axial_DIN0207 series, Axial, Horizontal, pin pitch=7.62mm, 0.25W = 1/4W, length*diameter=6.3*2.5mm^2, http://cdn-reichelt.de/documents/datenblatt/B400/1_4W%23YAG.pdf")
     (tags "Resistor Axial_DIN0207 series Axial Horizontal pin pitch 7.62mm 0.25W = 1/4W length 6.3mm diameter 2.5mm")
-    (property "Sheetfile" "C:/programming_land/kicad_projects/kp_espixelstick/espixelstick/espixelstick.sch")
+    (property "Sheetfile" "espixelstick.kicad_sch")
     (property "Sheetname" "")
     (property "ki_description" "Resistor, small symbol")
@@
     (descr "Resistor, Axial_DIN0207 series, Axial, Horizontal, pin pitch=7.62mm, 0.25W = 1/4W, length*diameter=6.3*2.5mm^2, http://cdn-reichelt.de/documents/datenblatt/B400/1_4W%23YAG.pdf")
     (tags "Resistor Axial_DIN0207 series Axial Horizontal pin pitch 7.62mm 0.25W = 1/4W length 6.3mm diameter 2.5mm")
-    (property "Sheetfile" "C:/programming_land/kicad_projects/kp_espixelstick/espixelstick/espixelstick.sch")
+    (property "Sheetfile" "espixelstick.kicad_sch")
     (property "Sheetname" "")
     (property "ki_description" "Resistor, small symbol")
@@
     (descr "TO-220-3, Vertical, RM 2.54mm")
     (tags "TO-220-3 Vertical RM 2.54mm")
-    (property "Sheetfile" "C:/programming_land/kicad_projects/kp_espixelstick/espixelstick/espixelstick.sch")
+    (property "Sheetfile" "espixelstick.kicad_sch")
     (property "Sheetname" "")
     (property "ki_description" "800mA Fixed Low Drop Positive Voltage Regulator, Fixed Output 3.3V, SOT-223")
